File: header.sch (KiCad schematic (older format))
At the start: 47 parts, among them J1 Conn_01x10, J2 Conn_01x08, J3 Conn_01x06, J4 Conn_01x08, Q2 Q_NMOS_GSD, Q3 Q_NMOS_GSD, Q4 Q_NMOS_GSD, SW6 SW_Push, U1 ICE40HX4K-TQ144, U20 MAX11614, U22 MAX40200AUK, U23 MAX40200AUK, U8 TXS0108EPW, U9 TXS0108EPW, Y2 ECS-3225S33-500-FN-TR

Commit message: More complete BOM
Parts:
- C87, C88, C91, C92: Description CAP CER 10UF 6.3V X5R 0603 -> CAP CER 10UF 6.3V X5R 0603
- D17: Description (none) -> LED RED DIFFUSED 1608 SMD; Digikey (none) -> SML-D12U1WT86CT-ND; Mfg Name (none) -> Rohm Semiconductor; Mfg Part Num (none) -> SML-D12U1WT86; Spec (none) -> Any
- J1: Description (none) -> CONN HDR 10POS 0.1 GOLD PCB; Digikey (none) -> 732-2859-ND; Mfg Name (none) -> Wurth Electronics Inc.; Mfg Part Num (none) -> 61301011821; Spec (none) -> Any
- J2, J4: Description (none) -> CONN HDR 8POS 0.1 GOLD PCB; Digikey (none) -> S7041-ND; Mfg Name (none) -> Sullins Connector Solutions; Mfg Part Num (none) -> PPPC081LFBN-RC; Spec (none) -> Any
- J3: Description (none) -> CONN HDR 6POS 0.1 GOLD PCB; Digikey (none) -> S7039-ND; Mfg Name (none) -> Sullins Connector Solutions; Mfg Part Num (none) -> PPPC061LFBN-RC; Spec (none) -> Any
- PMOD1, PMOD2, PMOD3: Description (none) -> CONN HDR 12POS 0.1 GOLD PCB R/A; Digikey (none) -> S5559-ND; Mfg Name (none) -> Sullins Connector Solutions; Mfg Part Num (none) -> PPPC062LJBN-RC; Spec (none) -> Any
- R31, R32, R61, R62, R63, R64: Description (none) -> RES 4.7K OHM 5% 1/10W 0603; Digikey (none) -> RMCF0603JT4K70CT-ND; Mfg Name (none) -> Stackpole Electronics Inc; Mfg Part Num (none) -> RMCF0603JT4K70; Spec (none) -> Any
- R54, R71: Description (none) -> RES 10K OHM 5% 1/10W 0603; Digikey (none) -> RMCF0603JT10K0CT-ND; Mfg Name (none) -> Stackpole Electronics Inc; Mfg Part Num (none) -> RMCF0603JT10K0; Spec (none) -> Any
- R55: Description (none) -> RES SMD 270K OHM 1% 1/10W 0603; Digikey (none) -> 311-270KHRCT-ND; Mfg Name (none) -> Yageo; Mfg Part Num (none) -> RC0603FR-07270KL; Spec (none) -> Any
- R60: Description (none) -> RES 560 OHM 5% 1/8W 0603; Digikey (none) -> 2019-RK73B1JTTD561JCT-ND; Mfg Name (none) -> KOA Speer Electronics, Inc.; Mfg Part Num (none) -> RK73B1JTTD561J; Spec (none) -> Any
- R69: Description (none) -> RES SMD 30K OHM 1% 1/10W 0603; Digikey (none) -> 311-30.0KHRCT-ND; Mfg Name (none) -> Yageo; Mfg Part Num (none) -> RC0603FR-0730KL; Spec (none) -> Any
- R70: Description (none) -> RES SMD 1K OHM 5% 1/10W 0603; Digikey (none) -> 311-1.0KGRCT-ND; Mfg Name (none) -> Yageo; Mfg Part Num (none) -> RC0603JR-071KL; Spec (none) -> Any
