File: ui.sch (KiCad schematic (older format))
At the start: 45 parts, among them SW1 SW_Push, SW2 SW_Push, SW3 SW_Push, SW4 SW_Push, SW5 SW_Push, SW8 JS202011SCQN, SW9 JS202011SCQN, U1 ICE40HX4K-TQ144

Commit message: More complete BOM
Parts:
- D1, D2, D3, D4, D5, D6, D7, D8: Description (none) -> LED RED DIFFUSED 1608 SMD; Digikey (none) -> SML-D12U1WT86CT-ND; Mfg Name (none) -> Rohm Semiconductor; Mfg Part Num (none) -> SML-D12U1WT86; Spec (none) -> Any
- R1, R2, R3, R4, R5, R6, R7, R8: Description (none) -> RES 560 OHM 5% 1/8W 0603; Digikey (none) -> 2019-RK73B1JTTD561JCT-ND; Mfg Name (none) -> KOA Speer Electronics, Inc.; Mfg Part Num (none) -> RK73B1JTTD561J; Spec (none) -> Any
- R10, R11, R12, R13, R50, R51, R9: Description (none) -> RES 4.7K OHM 5% 1/10W 0603; Digikey (none) -> RMCF0603JT4K70CT-ND; Mfg Name (none) -> Stackpole Electronics Inc; Mfg Part Num (none) -> RMCF0603JT4K70; Spec (none) -> Any
- R24, R25, R26, R27, R28, R56, R57: Description (none) -> RES 470 OHM 5% 1/10W 0603; Digikey (none) -> RMCF0603JT470RCT-ND; Mfg Name (none) -> Stackpole Electronics Inc; Mfg Part Num (none) -> RMCF0603JT470R; Spec (none) -> Any
